Commit message: 新文件：   .vscode/c_cpp_properties.json 	新文件：   .vscode/settings.json 	修改：     doc/ethercat_driver_doc.md 	修改：     src/ethercat_device_control/include/ethercat_device_control/ethercat_hardware_interface.hpp 	修改：     src/ethercat_device_control/launch/ethercat_bringup.launch.py 	修改：     src/ethercat_device_control/src/ethercat_hardware_interface.cpp 	新文件：   src/rm_force_publisher/README.md 	新文件：   src/rm_force_publisher/config/force_calibration.yaml 	新文件：   src/rm_force_publisher/launch/force_publisher.launch.py 	新文件：   src/rm_force_publisher/package.xml 	新文件：   src/rm_force_publisher/resource/rm_force_publisher 	新文件：   src/rm_force_publisher/rm_force_publisher/__init__.py 	新文件：   src/rm_force_publisher/rm_force_publisher/force_publisher_node.py 	新文件：   src/rm_force_publisher/setup.cfg 	新文件：   src/rm_force_publisher/setup.py 	新文件：   src/rm_hardware_interface/CMakeLists.txt 	新文件：   src/rm_hardware_interface/include/rm_hardware_interface/rm_hardware_interface.hpp 	新文件：   src/rm_hardware_interface/package.xml 	新文件：   src/rm_hardware_interface/rm_hardware_interface.xml 	新文件：   src/rm_hardware_interface/src/rm_hardware_interface.cpp 	修改：     src/robot_new_moveit/config/robot_new.ros2_control.xacro 	修改：     src/robot_new_moveit/config/ros2_controllers.yaml 	修改：     src/ros2_rm_robot-humble/rm_driver/config/rm_75_config.yaml 	修改：     src/ros2_rm_robot-humble/rm_driver/launch/rm_65_driver.launch.py 	修改：     src/ros2_rm_robot-humble/rm_driver/launch/rm_75_driver.launch.py 	新文件：   start_robot.sh

File: src/robot_new_moveit/config/robot_new.ros2_control.xacro (robot description, xacro)
@@ -2,10 +2,12 @@
 <robot xmlns:xacro="http://www.ros.org/wiki/xacro">
     <xacro:macro name="robot_new_ros2_control" params="name initial_positions_file">
-        <xacro:property name="initial_positions" value="${load_yaml(initial_positions_file)['initial_positions']}"/>
-        <ros2_control name="${name}" type="system">
+        <xacro:property name="initial_positions" value="${xacro.load_yaml(initial_positions_file)['initial_positions']}"/>
+        <!-- EtherCAT System: Controls the 5 custom motors -->
+        <ros2_control name="EthercatSystem" type="system">
             <hardware>
                 <plugin>ethercat_device_control/EthercatHardwareInterface</plugin>
                 <param name="use_dummy_mode">false</param>
             </hardware>
+            <!-- Slave 0: Straight Joint (Participates in motion planning) -->
             <joint name="straight_joint">
                 <command_interface name="position"/>
@@ -16,4 +18,55 @@
                 <state_interface name="velocity"/>
             </joint>
+            <!-- Slave 1: Front Wheel -->
+            <joint name="front_wheel_joint">
+                <command_interface name="position"/>
+                <command_interface name="velocity"/>
+                <command_interface name="effort"/>
+                <state_interface name="position">
+                  <param name="initial_value">0.0</param>
+                </state_interface>
+                <state_interface name="velocity"/>
+                <state_interface name="effort"/>
+            </joint>
+            <!-- Slave 2: Rear Wheel -->
+            <joint name="rear_wheel_joint">
+                <command_interface name="position"/>
+                <command_interface name="velocity"/>
+                <command_interface name="effort"/>
+                <state_interface name="position">
+                  <param name="initial_value">0.0</param>
+                </state_interface>
+                <state_interface name="velocity"/>
+                <state_interface name="effort"/>
+            </joint>
+            <!-- Slave 3: Rear Clamp Wheel -->
+            <joint name="rear_clamp_wheel_joint">
+                <command_interface name="position"/>
+                <command_interface name="velocity"/>
+                <command_interface name="effort"/>
+                <state_interface name="position">
+                  <param name="initial_value">0.0</param>
+                </state_interface>
+                <state_interface name="velocity"/>
+                <state_interface name="effort"/>
+            </joint>
+            <!-- Slave 4: Front Clamp Wheel -->
+            <joint name="front_clamp_wheel_joint">
+                <command_interface name="position"/>
+                <command_interface name="velocity"/>
+                <command_interface name="effort"/>
+                <state_interface name="position">
+                  <param name="initial_value">0.0</param>
+                </state_interface>
+                <state_interface name="velocity"/>
+                <state_interface name="effort"/>
+            </joint>
+        </ros2_control>
+        <!-- RealMan System: Controls the robotic arm -->
+        <ros2_control name="RealManSystem" type="system">
+            <hardware>
+                <!-- Use the newly created RealMan hardware interface -->
+                <plugin>rm_hardware_interface/RmHardwareInterface</plugin>
+            </hardware>
             <joint name="joint_1">
                 <command_interface name="position"/>
@@ -80,44 +133,4 @@
                 <state_interface name="velocity"/>
             </joint>
-            <joint name="front_wheel_joint">
-                <command_interface name="position"/>
-                <command_interface name="velocity"/>
-                <command_interface name="effort"/>
-                <state_interface name="position">
-                  <param name="initial_value">0.0</param>
-                </state_interface>
-                <state_interface name="velocity"/>
-                <state_interface name="effort"/>
-            </joint>
-            <joint name="rear_wheel_joint">
-                <command_interface name="position"/>
-                <command_interface name="velocity"/>
-                <command_interface name="effort"/>
-                <state_interface name="position">
-                  <param name="initial_value">0.0</param>
-                </state_interface>
-                <state_interface name="velocity"/>
-                <state_interface name="effort"/>
-            </joint>
-            <joint name="front_clamp_wheel_joint">
-                <command_interface name="position"/>
-                <command_interface name="velocity"/>
-                <command_interface name="effort"/>
-                <state_interface name="position">
-                  <param name="initial_value">0.0</param>
-                </state_interface>
-                <state_interface name="velocity"/>
-                <state_interface name="effort"/>
-            </joint>
-            <joint name="rear_clamp_wheel_joint">
-                <command_interface name="position"/>
-                <command_interface name="velocity"/>
-                <command_interface name="effort"/>
-                <state_interface name="position">
-                  <param name="initial_value">0.0</param>
-                </state_interface>
-                <state_interface name="velocity"/>
-                <state_interface name="effort"/>
-            </joint>
         </ros2_control>
     </xacro:macro>
